Commit message: clean up code

File: catkin_ws/src/simulation/walker_description/urdf/accessories/webcam_c930e.urdf.xacro (robot description, xacro)
@@ -34,5 +34,5 @@
         <gazebo reference="${frame}_link">
             <sensor type="camera" name="camera1">
-                <visualize>true</visualize>
+                <!-- <visualize>true</visualize> -->
                 <update_rate>${update_rate}</update_rate>
                 <camera name="head">

File: catkin_ws/src/simulation/walker_description/urdf/walker.urdf.xacro (robot description, xacro)
@@ -159,5 +159,5 @@
         </collision>
     </link>
-    <joint name="force_sensor_joint" type="revolute"> <!-- fixed -->
+    <joint name="force_sensor_joint" type="fixed"> <!-- revolute -->
         <origin xyz="0.16109 0 0.81585" rpy="0 0 -1.5708" />
         <parent link="base_link" />
