Commit message: add sensor mount in simulation

File: catkin_ws/src/simulation/walker_description/urdf/walker.urdf.xacro (robot description, xacro)
@@ -275,3 +275,31 @@
         <child link="camera_link" />
     </joint>
+    <!-- Sensor mount -->
+    <link name='sensor_mount_link'>
+        <inertial>
+            <origin xyz="0.1 0 0" rpy="0 0 0" />
+            <mass value="0.1" />
+            <box_inertia m="0.1" x="0.2" y="0.08" z="0.01"/>
+        </inertial>
+        <collision name='collision'>
+            <origin xyz="0.1 0 0" rpy="0 0 0" />
+            <geometry>
+                <box size="0.2 0.08 0.01" />
+            </geometry>
+        </collision>
+        <visual name='visual'>
+            <origin xyz="0.1 0 0" rpy="0 0 0" />
+            <geometry>
+                <box size="0.2 0.08 0.01" />
+            </geometry>
+            <material name="">
+                <color rgba="0.79216 0.81961 0.93333 1" />
+            </material>
+        </visual>
+    </link>
+    <joint name="sensor_mount_joint" type="fixed">
+        <origin xyz="0.24 0 0.535" rpy="0 0 0" />
+        <parent link="base_link"/>
+        <child link="sensor_mount_link"/>
+    </joint>
 </robot>

Commit message: rename robotnamespace

File: catkin_ws/src/simulation/walker_description/urdf/walker.urdf.xacro (robot description, xacro)
@@ -1,6 +1,6 @@
 <?xml version="1.0" encoding="UTF-8"?>
-<robot name="active_walker" xmlns:xacro="http://ros.org/wiki/xacro">
+<robot name="walker" xmlns:xacro="http://ros.org/wiki/xacro">
     <!-- <xacro:arg name="robot_namespace" default="/" />  -->
-    <xacro:arg name="robot_namespace" default="active_walker" />
+    <xacro:arg name="robot_namespace" default="walker" />
     <!-- Included URDF/XACRO Files -->
     <xacro:include filename="$(find walker_description)/urdf/accessories/webcam_c930e.urdf.xacro"/>
@@ -92,5 +92,5 @@
         <axis xyz="0 0 1" />
         <!-- <dynamics friction="0.001" /> -->
-        <joint_properties damping="0.0" friction="0.0"/>
+        <joint_properties damping="1.0" friction="0.0"/>
         <limit effort="100" velocity="100"/>
     </joint>
@@ -130,5 +130,5 @@
         <!-- <limit lower="0" upper="0" effort="0" velocity="0" /> -->
         <!-- <dynamics friction="0.001" /> -->
-        <joint_properties damping="0.0" friction="0.0"/>
+        <joint_properties damping="1.0" friction="0.0"/>
         <limit effort="100" velocity="100"/>
     </joint>
@@ -164,7 +164,8 @@
         <child link="force_sensor_link" />
         <axis xyz="0 0 1" />
-        <limit lower="0" velocity="1000" upper="0" effort="1000" />
+        <limit lower="0" velocity="100" upper="0" effort="100" />
         <!-- <safety_controller k_velocity="10" k_position="15" soft_lower_limit="-2.0" soft_upper_limit="0.5" />
         <dynamics damping="0.0" friction="0.0"/> -->
+        <dynamics damping="0.0" friction="0.0"/>
     </joint>
     <!-- Handrail link -->
@@ -193,9 +194,11 @@
         </collision>
     </link>
-    <joint name="handrail_joint" type="fixed">
+    <joint name="handrail_joint" type="fixed"> <!-- revolute -->
         <origin xyz="0 0 0.0565" rpy="0 0 1.5708" />
         <parent link="force_sensor_link" />
         <child link="handrail_link" />
-        <axis xyz="0 0 0" />
+        <axis xyz="0 0 1" />
+        <limit lower="0" velocity="100" upper="0" effort="100" />
+        <dynamics damping="1.0"/>
     </joint>
     <!-- Front right caster wheel link & joint-->

Commit message: add estop gz model, modify social agf function, clean up agf vis code, and clean up subgoal generating code

File: catkin_ws/src/simulation/walker_description/urdf/walker.urdf.xacro (robot description, xacro)
@@ -6,4 +6,5 @@
     <xacro:include filename="$(find walker_description)/urdf/accessories/webcam_c930e.urdf.xacro"/>
     <xacro:include filename="$(find walker_description)/urdf/accessories/ydlidar_g4.urdf.xacro" />
+    <xacro:include filename="$(find walker_description)/urdf/accessories/estop.urdf.xacro" />
     <!-- Gazebo plugin -->
     <xacro:include filename="$(find walker_description)/urdf/walker.gazebo" />
@@ -306,3 +307,10 @@
         <child link="sensor_mount_link"/>
     </joint>
+    <!-- E-stop -->
+    <estop frame="estop" />
+    <joint name="estop_joint1" type="fixed">
+        <origin xyz="0.161 0 0.905" rpy="0 0 0" />
+        <parent link="base_link" />
+        <child link="estop_base" />
+    </joint>
 </robot>
